File: hardware/presto-jr-v2.0/led_interface.kicad_sch (KiCad schematic)
At the start: 8 parts

Commit message: updated v2
Parts:
- removed D701, D702, D703, D704: LED, LED_SMD:LED_1206_3216Metric_Pad1.42x1.75mm_HandSolder, symbol Device:LED
- removed R701, R702, R703, R704: RES, Resistor_SMD:R_1206_3216Metric_Pad1.30x1.75mm_HandSolder, symbol Device:R_US
- added D2: LED, symbol Device:LED
- added Q2: BC337, Package_TO_SOT_THT:TO-92_Inline, symbol Transistor_BJT:BC337
- added R1, R2: R_US, symbol Device:R_US
- added U2: PC817, Package_DIP:DIP-4_W7.62mm, symbol Isolator:PC817
Connections:
- net RED_IN: now also Q2.1 (C)
- new net: Q2.2 (B), R2.2
- new net: R1.2, U2.1
- new net: D2.2 (A), U2.2
- new net: R2.1, U2.3
- new net 5V_LED: U2.4
- new net LED_GND: Q2.3 (E)
Other:
- note added: "3.3V: 300 Ohm 5V: 550 Ohm 1k?"
- note added: "Fwd V 1.2-1.4V"
- note added: "LOAD HI"
- note added: "LOAD LO"
- note added: "LOAD OUT"
- note added: "Light Tower 120mA per color at 12V"

Commit message: added presto jr
Parts:
- added D702, D703, D704: LED, LED_SMD:LED_1206_3216Metric_Pad1.42x1.75mm_HandSolder, symbol Device:LED
- added JP701: LED_SHARE_5V, Jumper:SolderJumper-2_P1.3mm_Open_RoundedPad1.0x1.5mm, symbol Jumper:SolderJumper_2_Open
- added Q701, Q702, Q703: BC337, Package_TO_SOT_THT:TO-92_Inline, symbol Transistor_BJT:BC337
- added R701, R702, R707, R708: 100R, Resistor_SMD:R_1206_3216Metric_Pad1.30x1.75mm_HandSolder, symbol Device:R_US
- added R703, R704, R709: 300R, Resistor_SMD:R_1206_3216Metric_Pad1.30x1.75mm_HandSolder, symbol Device:R_US
- added R705, R706, R711: 600R, Resistor_SMD:R_1206_3216Metric_Pad1.30x1.75mm_HandSolder, symbol Device:R_US
- added U701: L7805, Package_TO_SOT_THT:TO-220-3_Horizontal_TabDown, symbol Regulator_Linear:L7805
- added U703, U704, U705: PC817, Package_DIP:DIP-4_W7.62mm, symbol Isolator:PC817
- D701: renamed from D2; footprint (none) -> LED_SMD:LED_1206_3216Metric_Pad1.42x1.75mm_HandSolder
- R710: renamed from R1; value R_US -> 300R; footprint (none) -> Resistor_SMD:R_1206_3216Metric_Pad1.30x1.75mm_HandSolder
- R712: renamed from R2; value R_US -> 600R; footprint (none) -> Resistor_SMD:R_1206_3216Metric_Pad1.30x1.75mm_HandSolder
- renumbered Q2 to Q704, U2 to U702
Connections:
- net 5V_LED: now also JP701.1 (A), U701.3 (OUT), U703.4, U704.4, U705.4
- net BLU_IN: now also Q704.1 (C)
- net GRN_IN: now also Q703.1 (C)
- net LED_GND: now also Q701.3 (E), Q702.3 (E), Q703.3 (E), U701.2 (GND)
- net RED_IN: now also Q701.1 (C); no longer Q704.1 (C)
- net YEL_IN: now also Q702.1 (C)
- net at U702.1: now also R703.2; no longer R710.2
- net at D701.2 (A): now also R701.2; no longer U702.2
- net at U702.3: now also R705.1; no longer R712.1
- net GND: now reaches D701.1 (K)
- net GND: now also U702.2, D702.1 (K), D703.1 (K), D704.1 (K), U703.2, U704.2, U705.2
- net BLU_SIG: now reaches R710.1
- net BLU_SIG: now also R708.1
- new net: Q702.2 (B), R706.2
- new net: D703.2 (A), R707.2
- new net: R704.2, U703.1
- new net: D704.2 (A), R708.2
- new net: R711.1, U704.3
- new net: Q703.2 (B), R711.2
- new net: R706.1, U703.3
- new net: R709.2, U704.1
- new net: D702.2 (A), R702.2
- new net: R710.2, U705.1
- new net: R712.1, U705.3
- new net: Q701.2 (B), R705.2
- new net +5V: JP701.2 (B)
- new net GRN_SIG: R707.1, R709.1
- new net LED_PWR_IN: U701.1 (IN)
- new net RED_SIG: R701.1, R703.1
- new net YEL_SIG: R702.1, R704.1
Other:
- note added: "3.3V"
- note added: "3.3V: 300 Ohm 5V: 550 Ohm"
- note added: "5V"
- note added: "GND"
- note added: "Indicator"
- note added: "LED"
- note added: "LED GND"
- note added: "Max 35V"
- note added: "Summary: The PC817 optocoupler is used to isolate the external light circuit from the main board. The BC337 NPN BJT was chosen due to its robust characteristics, but a 2N3904 could potentially suffice given low current. R1 regulates current for the PC817 LED, calculated based on an assumption of a forward voltage of 1.2V and a forward current of 7mA. R2 ensures saturation of the BJT. The PC817 ha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"
- note removed: "3.3V: 300 Ohm 5V: 550 Ohm 1k?"
- note removed: "LOAD HI"
- note removed: "LOAD LO"
- note removed: "LOAD OUT"
- moved on the sheet: D701, Q704, R710, R712, U702
