File: hardware/presto-jr-v2.0/presto-jr-v2.0.kicad_pcb (KiCad board)
At the start: 2 copper layers, 95.5 x 100.5 mm, 43 parts, among them J1 Conn_01x03_Pin, J101 12V IN, J102 Conn_01x02_Pin, J4 E-Stop, J5 E-Stop, J701 LED Connector, K301 12V SRD Form C, K401 12V SRD Form C

Commit message: updated v2
Parts:
- removed J102: Conn_01x02_Pin, Connector_JST:JST_XH_B2B-XH-A_1x02_P2.50mm_Vertical
- removed J701: LED Connector, Connector_JST:JST_XH_B5B-XH-A_1x05_P2.50mm_Vertical
- added J10: Conn_01x04_Pin, Connector_JST:JST_XH_S4B-XH-SM4-TB_1x04-1MP_P2.50mm_Horizontal, B.Cu at (105.7, 38.8)
- added J11: Conn_01x04_Pin, Connector_JST:JST_XH_S4B-XH-SM4-TB_1x04-1MP_P2.50mm_Horizontal, F.Cu at (88.8, 38.8)
- added J12: Conn_01x04_Pin, Connector_JST:JST_XH_S4B-XH-SM4-TB_1x04-1MP_P2.50mm_Horizontal, B.Cu at (88.8, 38.8)
- added J2: LED CONN, Connector_JST:JST_XH_S8B-XH-A_1x08_P2.50mm_Horizontal, F.Cu at (152.8, 42.0)
- added J7: Conn_01x04_Pin, Connector_JST:JST_XH_S4B-XH-SM4-TB_1x04-1MP_P2.50mm_Horizontal, F.Cu at (122.5, 38.8)
- added J8: Conn_01x04_Pin, Connector_JST:JST_XH_S4B-XH-SM4-TB_1x04-1MP_P2.50mm_Horizontal, B.Cu at (122.5, 38.8)
- added J9: Conn_01x04_Pin, Connector_JST:JST_XH_S4B-XH-SM4-TB_1x04-1MP_P2.50mm_Horizontal, F.Cu at (105.7, 38.8)
- added JP106: LED_SHARE_5V, Jumper:SolderJumper-2_P1.3mm_Open_RoundedPad1.0x1.5mm, F.Cu at (158.5, 139.6)
- added JP107: LED_SHARE_GND, Jumper:SolderJumper-2_P1.3mm_Open_RoundedPad1.0x1.5mm, F.Cu at (172.7, 138.2)
- added Q2: BC337, Package_TO_SOT_THT:TO-92_Inline, F.Cu at (165.6, 157.1)
- added U2: PC817, Package_DIP:DIP-4_W7.62mm, F.Cu at (136.5, 138.4)
- A101: footprint Module:RaspberryPi_Pico_Common_Unspecified -> Module:RaspberryPi_Pico_SMD_HandSolder
- A601, D101: moved to B.Cu
- moved F1 119.6 mm to (51.9, 133.8)
- moved A601 63.8 mm to (89.7, 114.7), turned to 90 degrees
- moved D101 55.4 mm to (80.5, 130.4)
- moved J101 36.0 mm to (83.4, 136.7), turned to 180 degrees
- moved A101 19.6 mm to (105.4, 110.8)
- moved J4 18.1 mm to (140.6, 144.0)
- moved J5 18.1 mm to (140.6, 144.0)
- moved J1 18.0 mm to (122.2, 144.0)
Connections:
- A101 pad 25: Net-(A101-GPIO19) -> unconnected-(A101-GPIO19-Pad25)
- A101 pad 26: Net-(A101-GPIO20) -> unconnected-(A101-GPIO20-Pad26)
- A101 pad 29: Net-(A101-GPIO22) -> unconnected-(A101-GPIO22-Pad29)
- A101 pad 34: Net-(A101-GPIO28_ADC2) -> unconnected-(A101-GPIO28_ADC2-Pad34)
- J5 pad 6: /ESTOP_IN -> unconnected-(J5-Pin_6-Pad6)
Routing:
- net +5V: track 0.00 -> 38.5 mm, vias 0 -> 1
- net +12V: track 0.00 -> 16.4 mm
- net +BATT: track 0.00 -> 7.17 mm
Other:
- board size 95.5 x 100.5 mm -> 80 x 95 mm

Commit message: added presto jr
Parts:
- removed J2: LED CONN, Connector_JST:JST_XH_S8B-XH-A_1x08_P2.50mm_Horizontal
- removed JP103: ch6 to estop, Jumper:SolderJumper-2_P1.3mm_Open_RoundedPad1.0x1.5mm
- removed JP104, JP105: RC PWR, Jumper:SolderJumper-2_P1.3mm_Open_RoundedPad1.0x1.5mm
- removed JP106: LED_SHARE_5V, Jumper:SolderJumper-2_P1.3mm_Open_RoundedPad1.0x1.5mm
- removed JP107: LED_SHARE_GND, Jumper:SolderJumper-2_P1.3mm_Open_RoundedPad1.0x1.5mm
- removed Q2: BC337, Package_TO_SOT_THT:TO-92_Inline
- removed the REF** at (59.6, 95.6)
- removed the REF** at (60.0, 90.6)
- removed TP3: TestPoint, TestPoint:TestPoint_THTPad_2.5x2.5mm_Drill1.2mm
- removed U2: PC817, Package_DIP:DIP-4_W7.62mm
- removed U3: ~, Package_DIP:DIP-14_W7.62mm_Socket_LongPads
- added J108: LED_CONN, Connector_JST:JST_XH_S5B-XH-A_1x05_P2.50mm_Horizontal, F.Cu at (137.5, 150.8)
- added JP701: LED_SHARE_5V, Jumper:SolderJumper-2_P1.3mm_Open_RoundedPad1.0x1.5mm, B.Cu at (144.8, 116.0)
- added Q701: BC337, Package_TO_SOT_THT:TO-92_Inline, F.Cu at (131.4, 141.6)
- added Q702: BC337, Package_TO_SOT_THT:TO-92_Inline, F.Cu at (138.9, 141.6)
- added Q703: BC337, Package_TO_SOT_THT:TO-92_Inline, F.Cu at (146.4, 141.6)
- added Q704: BC337, Package_TO_SOT_THT:TO-92_Inline, F.Cu at (153.9, 141.6)
- added R705: 600R, Resistor_SMD:R_1206_3216Metric_Pad1.30x1.75mm_HandSolder, B.Cu at (130.1, 134.6)
- added R706: 600R, Resistor_SMD:R_1206_3216Metric_Pad1.30x1.75mm_HandSolder, B.Cu at (137.6, 134.6)
- added R707: 100R, Resistor_SMD:R_1206_3216Metric_Pad1.30x1.75mm_HandSolder, F.Cu at (145.3, 125.2)
- added R708: 100R, Resistor_SMD:R_1206_3216Metric_Pad1.30x1.75mm_HandSolder, F.Cu at (152.8, 125.2)
- added R709: 300R, Resistor_SMD:R_1206_3216Metric_Pad1.30x1.75mm_HandSolder, F.Cu at (145.3, 128.1)
- added R710: 300R, Resistor_SMD:R_1206_3216Metric_Pad1.30x1.75mm_HandSolder, F.Cu at (152.8, 128.1)
- added R711: 600R, Resistor_SMD:R_1206_3216Metric_Pad1.30x1.75mm_HandSolder, B.Cu at (145.1, 134.6)
- added R712: 600R, Resistor_SMD:R_1206_3216Metric_Pad1.30x1.75mm_HandSolder, B.Cu at (152.6, 134.6)
- added REF**: MountingHole_2.7mm_M2.5, MountingHole:MountingHole_2.7mm_M2.5, F.Cu at (85.0, 155.0)
- added REF**: MountingHole_2.7mm_M2.5, MountingHole:MountingHole_2.7mm_M2.5, F.Cu at (155.0, 62.0)
- added REF**: MountingHole_2.7mm_M2.5, MountingHole:MountingHole_2.7mm_M2.5, F.Cu at (85.0, 62.0)
- added REF**: MountingHole_2.7mm_M2.5, MountingHole:MountingHole_2.7mm_M2.5, F.Cu at (155.0, 155.0)
- added TP103: TestPoint, TestPoint:TestPoint_THTPad_2.5x2.5mm_Drill1.2mm, F.Cu at (155.6, 99.1)
- added U701: L7805, Package_TO_SOT_THT:TO-220-3_Horizontal_TabDown, F.Cu at (136.3, 113.5)
- added U702: PC817, Package_DIP:DIP-4_W7.62mm, F.Cu at (131.4, 130.8)
- added U703: PC817, Package_DIP:DIP-4_W7.62mm, F.Cu at (138.9, 130.8)
- added U704: PC817, Package_DIP:DIP-4_W7.62mm, F.Cu at (146.4, 130.8)
- added U705: PC817, Package_DIP:DIP-4_W7.62mm, F.Cu at (153.9, 130.8)
- D301, D403, D701, D702, D703, D704, J101, R301: moved to B.Cu
- J102: renamed from J1; value Conn_01x03_Pin -> RC_ES
- J103: renamed from J4; moved to B.Cu
- J105: renamed from J7; value Conn_01x04_Pin -> IO01-02
- J106: renamed from J8; value Conn_01x04_Pin -> IO03-04; moved to F.Cu
- J107: renamed from J9; value Conn_01x04_Pin -> IO05-06
- J109: renamed from J10; value Conn_01x04_Pin -> IO07-08; moved to F.Cu
- J110: renamed from J11; value Conn_01x04_Pin -> IO09-10; footprint Connector_JST:JST_XH_S4B-XH-SM4-TB_1x04-1MP_P2.50mm_Horizontal -> Connector_JST:JST_XH_B4B-XH-A_1x04_P2.50mm_Vertical
- J111: renamed from J12; value Conn_01x04_Pin -> IO11-12; footprint Connector_JST:JST_XH_S4B-XH-SM4-TB_1x04-1MP_P2.50mm_Horizontal -> Connector_JST:JST_XH_B4B-XH-A_1x04_P2.50mm_Vertical; moved to F.Cu
- JP101: value ch6 to gpio16 -> RC PWR; moved to B.Cu
- JP102: value gpio16 to estop -> IO-CH-ES; footprint Jumper:SolderJumper-2_P1.3mm_Open_RoundedPad1.0x1.5mm -> Jumper:SolderJumper-3_P1.3mm_Bridged2Bar12_RoundedPad1.0x1.5mm; moved to B.Cu
- R701, R702: value 220 -> 100R
- R703, R704: value 220 -> 300R
- TP106: renamed from TP4; value TestPoint -> +5V
- TP107: renamed from TP5; value TestPoint -> +3V3
- moved D704 133.4 mm to (152.8, 126.4), turned to -90 degrees
- moved R702 130.9 mm to (137.8, 125.2)
- moved D703 130.0 mm to (145.3, 126.4), turned to -90 degrees
- moved R701 127.9 mm to (130.2, 125.2)
- moved R704 127.6 mm to (137.8, 128.1)
- moved D702 127.2 mm to (137.8, 126.4), turned to -90 degrees
- moved R703 124.6 mm to (130.2, 128.1)
- moved D701 124.5 mm to (130.2, 126.4), turned to -90 degrees
- moved TP106 90.1 mm to (84.4, 96.6), turned to 90 degrees
- moved J103 89.7 mm to (120.9, 56.5)
- moved D403 89.2 mm to (133.0, 89.3), turned to -90 degrees
- moved TP107 89.1 mm to (84.4, 101.5), turned to 90 degrees
- moved TP102 88.6 mm to (84.4, 91.7), turned to 90 degrees
- moved J104 87.5 mm to (142.6, 56.5), turned to 0 degrees
- moved D301 87.1 mm to (129.2, 89.3), turned to -90 degrees
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- renumbered F1 to F401, J5 to J104, TP1 to TP101, TP2 to TP102, TP7 to TP104, TP8 to TP105
Connections:
- net /EStop Reading/estop_signal renamed /io18
- net /gpio17 renamed /io17
- A101 pad 10: unconnected-(A101-GPIO7-Pad10) -> /io07
- A101 pad 11: unconnected-(A101-GPIO8-Pad11) -> /io08
- A101 pad 12: unconnected-(A101-GPIO9-Pad12) -> /io09
- A101 pad 14: unconnected-(A101-GPIO10-Pad14) -> /io10
- A101 pad 15: /CH1 -> /io11
- A101 pad 16: /CH2 -> /io12
- A101 pad 17: /CH3 -> unconnected-(A101-GPIO13-Pad17)
- A101 pad 19: /CH4 -> unconnected-(A101-GPIO14-Pad19)
- A101 pad 2: unconnected-(A101-GPIO1-Pad2) -> /io01
- A101 pad 20: /CH5 -> unconnected-(A101-GPIO15-Pad20)
- A101 pad 21: /gpio16 -> /io16
- A101 pad 25: unconnected-(A101-GPIO19-Pad25) -> /red_sig
- A101 pad 26: unconnected-(A101-GPIO20-Pad26) -> /yel_sig
- A101 pad 27: unconnected-(A101-GPIO21-Pad27) -> /grn_sig
- A101 pad 29: unconnected-(A101-GPIO22-Pad29) -> /blu_sig
- A101 pad 4: unconnected-(A101-GPIO2-Pad4) -> /io02
- A101 pad 5: unconnected-(A101-GPIO3-Pad5) -> /io03
- A101 pad 6: unconnected-(A101-GPIO4-Pad6) -> /io04
- A101 pad 7: unconnected-(A101-GPIO5-Pad7) -> /io05
- A101 pad 9: unconnected-(A101-GPIO6-Pad9) -> /io06
- A401 pad 10: +12V -> +BATT
- A401 pad 11: +12V -> +BATT
- A601 pad 2: +12V -> +BATT
- D101 pad 1: +12V -> +BATT
- D101 pad 2: +BATT -> Net-(D101-A)
- D403 pad 1: +12V -> +BATT
- D701 pad 1: Net-(D701-K) -> GND
- D701 pad 2: /LED Interface/red -> Net-(D701-A)
- D702 pad 1: Net-(D702-K) -> GND
- D702 pad 2: /LED Interface/yellow -> Net-(D702-A)
- D703 pad 1: Net-(D703-K) -> GND
- D703 pad 2: /LED Interface/green -> Net-(D703-A)
- D704 pad 1: Net-(D704-K) -> GND
- D704 pad 2: /LED Interface/blue -> Net-(D704-A)
- J101 pad 2: +BATT -> Net-(D101-A)
- J102 pad 2: Net-(J1-Pin_2) -> Net-(J102-Pin_2)
- J105 pad 2: /IO01 -> /io02
- J105 pad 4: /IO02 -> /io01
- J106 pad 2: /IO03 -> /io04
- J106 pad 4: /IO04 -> /io03
- J107 pad 2: /IO05 -> /io06
- J107 pad 4: /IO06 -> /io05
- J109 pad 2: /IO07 -> /io08
- J109 pad 4: /IO08 -> /io07
- J110 pad 2: /IO09 -> /io10
- J110 pad 4: /IO10 -> /io09
- J111 pad 2: /IO11 -> /io12
- J111 pad 4: /IO12 -> /io11
- JP101 pad 1: /ESTOP_CH -> +5V
- JP101 pad 2: /gpio16 -> Net-(J102-Pin_2)
- JP102 pad 1: /gpio16 -> /EStop Trigger/RC_IN
- JP102 pad 2: /EStop Trigger/RC_IN -> /ESTOP_CH
- K401 pad 5: +12V -> +BATT
- R701 pad 1: Net-(D701-K) -> /red_sig
- R701 pad 2: GND -> Net-(D701-A)
- R702 pad 1: Net-(D702-K) -> /yel_sig
- R702 pad 2: GND -> Net-(D702-A)
- R703 pad 1: Net-(D703-K) -> /red_sig
- R703 pad 2: GND -> Net-(R703-Pad2)
- R704 pad 1: Net-(D704-K) -> /yel_sig
- R704 pad 2: GND -> Net-(R704-Pad2)
Routing:
- net +BATT: track 7.17 -> 223.0 mm
- net +3V3: track 0.00 -> 180.7 mm, vias 0 -> 3
- net +5V: track 38.5 -> 183.9 mm, vias 1 -> 4
- net /io08: track 0.00 -> 142.9 mm, vias 0 -> 2
- net /io07: track 0.00 -> 137.8 mm, vias 0 -> 2
- net /io05: track 0.00 -> 128.1 mm, vias 0 -> 2
- net /io06: track 0.00 -> 127.9 mm, vias 0 -> 2
- net /ESTOP_COM: track 0.00 -> 119.5 mm, vias 0 -> 2
- net /io04: track 0.00 -> 118.4 mm, vias 0 -> 2
- net /io16: track 0.00 -> 117.5 mm, vias 0 -> 3
- net /ESTOP_IN: track 0.00 -> 112.7 mm, vias 0 -> 2
- net /io03: track 0.00 -> 112.6 mm, vias 0 -> 2
- net /io02: track 0.00 -> 101.6 mm, vias 0 -> 2
- net /io01: track 0.00 -> 101.2 mm, vias 0 -> 2
- net /EStop Trigger/RC_IN: track 0.00 -> 100.0 mm
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- added copper zone on B.Cu, net GND
Other:
- board size 80 x 95 mm -> 80 x 110 mm
- board text added: "+3V3"
- board text added: "+5V"
- board text added: "01 G 02 G"
- board text added: "03 G 04 G"
- board text added: "05 G 06 G"
- board text added: "07 G 08 G"
- board text added: "09 G 10 G"
- board text added: "11 G 12 G"
- board text added: "5 4 3 2 1 B G Y R V | | | | |"
- board text added: "5V to RC"
- board text added: "BATT"
- board text added: "ES|CH|IO16"
- board text added: "GND"
- board text added: "IF REG MISSING SEE REVERSE JP"
- board text added: "LED_CONN"
- board text added: "PRESTO v2.0r0"
- board text added: "RC_ES"
- board text added: "SHARE BOARD 5V WITH LED"
- board text added: "Sch Rev + Layout: S. Fish"
