File: hardware/presto-jr-v2.0/presto-jr-v2.0.kicad_pcb (KiCad board)
At the start: 2 copper layers, 80 x 110 mm, 64 parts, among them J101 12V IN, J102 RC_ES, J103 E-Stop, J104 E-Stop, J105 IO01-02, J106 IO03-04, J107 IO05-06, J108 LED_CONN, J109 IO07-08, J110 IO09-10, J111 IO11-12, K301 12V SRD Form C, K401 12V SRD Form C, Q701 BC337, Q702 BC337, Q703 BC337, Q704 BC337, U701 L7805, U702 PC817, U703 PC817, U704 PC817, U705 PC817

Commit message: I forget what I did
Parts:
- added JP103: EST-GND, Jumper:SolderJumper-2_P1.3mm_Bridged_RoundedPad1.0x1.5mm, B.Cu at (151.0, 76.8)
- J108: footprint Connector_JST:JST_XH_S5B-XH-A_1x05_P2.50mm_Horizontal -> GTMRG_Footprints:JST_XH_S5B-XH-SM4-TB_1x05-1MP_P2.50mm_Horizontal
- moved J108 5.55 mm to (142.0, 154.0)
- moved J102 0.90 mm to (125.0, 154.0)
Routing:
- net /ESTOP_COM: track 119.5 -> 144.8 mm
- net /ESTOP_IN: track 112.7 -> 97.6 mm, vias 2 -> 3
- net Net-(J102-Pin_2): track 5.58 -> 11.1 mm
- net /io11: track 79.0 -> 77.2 mm
- net /EStop Trigger/LOAD_LO: track 35.6 -> 37.3 mm
- net /io01: track 101.2 -> 102.3 mm
- net +3V3: track 180.7 -> 181.5 mm
- net /io12: track 84.7 -> 84.0 mm
- net +BATT: track 223.0 -> 222.3 mm
- net /LED Interface/YEL_IN: track 10.6 -> 9.92 mm
- net /LED Interface/RED_IN: track 14.7 -> 14.0 mm
- net /ESTOP_CH: track 6.90 -> 6.23 mm
- net GND: vias 211 -> 301
Other:
- board text added: "12-14V"
- board text added: "E C O C O C"
- board text added: "E-STOP JUNCTION"
- board text added: "E: Input O: Output C: Common Max Curr 3A"
- board text added: "PRIMARY"
- board text added: "SECONDARY"
- board text added: "X C O C O C"
