File: hardware/presto-jr-v2.0/presto-jr-v2.0.kicad_sch (KiCad schematic)
At the start: 21 parts, among them J1 Conn_01x03_Pin, J101 12V IN, J2 LED CONN, J4 E-Stop, J5 E-Stop

Commit message: updated v2
Parts:
- added J10, J11, J12, J7, J8, J9: Conn_01x04_Pin, Connector_JST:JST_XH_S4B-XH-SM4-TB_1x04-1MP_P2.50mm_Horizontal, symbol Connector:Conn_01x04_Pin
- A101: footprint Module:RaspberryPi_Pico_Common_Unspecified -> Module:RaspberryPi_Pico_SMD_HandSolder
- J2: footprint (none) -> Connector_JST:JST_XH_S8B-XH-A_1x08_P2.50mm_Horizontal
Connections:
- net GND: now also J10.1 (Pin_1), J10.3 (Pin_3), J11.1 (Pin_1), J11.3 (Pin_3), J12.1 (Pin_1), J12.3 (Pin_3), J7.1 (Pin_1), J7.3 (Pin_3), J8.1 (Pin_1), J8.3 (Pin_3), J9.1 (Pin_1), J9.3 (Pin_3)
- net GND_LED renamed LED_GND
- net V_LED renamed LED_V
- new net IO01: J7.2 (Pin_2)
- new net IO02: J7.4 (Pin_4)
- new net IO03: J8.2 (Pin_2)
- new net IO04: J8.4 (Pin_4)
- new net IO05: J9.2 (Pin_2)
- new net IO06: J9.4 (Pin_4)
- new net IO07: J10.2 (Pin_2)
- new net IO08: J10.4 (Pin_4)
- new net IO09: J11.2 (Pin_2)
- new net IO10: J11.4 (Pin_4)
- new net IO11: J12.2 (Pin_2)
- new net IO12: J12.4 (Pin_4)

Commit message: added presto jr
Parts:
- removed J2: LED CONN, Connector_JST:JST_XH_S8B-XH-A_1x08_P2.50mm_Horizontal, symbol Connector:Conn_01x08_Pin
- removed JP101: ch6 to gpio16, Jumper:SolderJumper-2_P1.3mm_Open_RoundedPad1.0x1.5mm, symbol Jumper:SolderJumper_2_Open
- removed JP102: gpio16 to estop, Jumper:SolderJumper-2_P1.3mm_Open_RoundedPad1.0x1.5mm, symbol Jumper:SolderJumper_2_Open
- removed JP103: ch6 to estop, Jumper:SolderJumper-2_P1.3mm_Open_RoundedPad1.0x1.5mm, symbol Jumper:SolderJumper_2_Open
- removed JP106: LED_SHARE_5V, Jumper:SolderJumper-2_P1.3mm_Open_RoundedPad1.0x1.5mm, symbol Jumper:SolderJumper_2_Open
- removed JP107: LED_SHARE_GND, Jumper:SolderJumper-2_P1.3mm_Open_RoundedPad1.0x1.5mm, symbol Jumper:SolderJumper_2_Open
- removed TP3: TestPoint, TestPoint:TestPoint_THTPad_2.5x2.5mm_Drill1.2mm, symbol Connector:TestPoint
- added J108: LED_CONN, Connector_JST:JST_XH_S5B-XH-A_1x05_P2.50mm_Horizontal, symbol Connector:Conn_01x05_Pin
- added JP102: IO-CH-ES, Jumper:SolderJumper-3_P1.3mm_Bridged2Bar12_RoundedPad1.0x1.5mm, symbol Jumper:SolderJumper_3_Bridged12
- J102: renamed from J1; value Conn_01x03_Pin -> RC_ES
- J105: renamed from J7; value Conn_01x04_Pin -> IO01-02
- J106: renamed from J8; value Conn_01x04_Pin -> IO03-04
- J107: renamed from J9; value Conn_01x04_Pin -> IO05-06
- J109: renamed from J10; value Conn_01x04_Pin -> IO07-08
- J110: renamed from J11; value Conn_01x04_Pin -> IO09-10; footprint Connector_JST:JST_XH_S4B-XH-SM4-TB_1x04-1MP_P2.50mm_Horizontal -> Connector_JST:JST_XH_B4B-XH-A_1x04_P2.50mm_Vertical
- J111: renamed from J12; value Conn_01x04_Pin -> IO11-12; footprint Connector_JST:JST_XH_S4B-XH-SM4-TB_1x04-1MP_P2.50mm_Horizontal -> Connector_JST:JST_XH_B4B-XH-A_1x04_P2.50mm_Vertical
- TP103: renamed from TP6; footprint (none) -> TestPoint:TestPoint_THTPad_2.5x2.5mm_Drill1.2mm
- TP106: renamed from TP4; value TestPoint -> +5V
- TP107: renamed from TP5; value TestPoint -> +3V3
- renumbered J4 to J103, J5 to J104, JP105 to JP101, TP1 to TP101, TP2 to TP102, TP7 to TP104, TP8 to TP105
Connections:
- net +12V is gone; now on net +BATT: D101.1 (K)
- net IO01 is gone; now on net io02: J105.2 (Pin_2)
- net IO02 is gone; now on net io01: J105.4 (Pin_4)
- net IO03 is gone; now on net io04: J106.2 (Pin_2)
- net IO04 is gone; now on net io03: J106.4 (Pin_4)
- net IO05 is gone; now on net io06: J107.2 (Pin_2)
- net IO06 is gone; now on net io05: J107.4 (Pin_4)
- net IO07 is gone; now on net io08: J109.2 (Pin_2)
- net IO08 is gone; now on net io07: J109.4 (Pin_4)
- net IO09 is gone; now on net io10: J110.2 (Pin_2)
- net IO10 is gone; now on net io09: J110.4 (Pin_4)
- net IO11 is gone; now on net io12: J111.2 (Pin_2)
- net IO12 is gone; now on net io11: J111.4 (Pin_4)
- net +BATT: now also J108.1 (Pin_1); no longer D101.2 (A), J101.2 (Pin_2)
- net ESTOP_CH: now also JP102.2 (C)
- net EStop Trigger/RC_IN: now also JP102.1 (A)
- net io07: now reaches A101.10 (GPIO7)
- net io08: now reaches A101.11 (GPIO8)
- net io09: now reaches A101.12 (GPIO9)
- net io10: now reaches A101.14 (GPIO10)
- net io01: now reaches A101.2 (GPIO1)
- net red_sig: now reaches A101.25 (GPIO19)
- net yel_sig: now reaches A101.26 (GPIO20)
- net grn_sig: now reaches A101.27 (GPIO21)
- net blu_sig: now reaches A101.29 (GPIO22)
- net io02: now reaches A101.4 (GPIO2)
- net io03: now reaches A101.5 (GPIO3)
- net io04: now reaches A101.6 (GPIO4)
- net io05: now reaches A101.7 (GPIO5)
- net io06: now reaches A101.9 (GPIO6)
- net CH1 renamed io11
- net CH2 renamed io12
- net CH3: no longer names the net of A101.17 (GPIO13)
- net CH4: no longer names the net of A101.19 (GPIO14)
- net CH5: no longer names the net of A101.20 (GPIO15)
- net EStop Reading/estop_signal renamed io18
- net gpio16 renamed io16
- net io16: now also JP102.3 (B)
- net gpio17 renamed io17
- new net: D101.2 (A), J101.2 (Pin_2)
- new net LED Interface/BLU_IN: J108.5 (Pin_5)
- new net LED Interface/GRN_IN: J108.4 (Pin_4)
- new net LED Interface/RED_IN: J108.2 (Pin_2)
- new net LED Interface/YEL_IN: J108.3 (Pin_3)
- no-connect marks 10 -> 13
Other:
- sheet LED Interface ports: added BLU_SIG, GRN_SIG, LED_GND_IN, LED_PWR_IN, RED_SIG, YEL_SIG; removed none
- note added: "E-Stop"
- note added: "IO"
- note added: "LED"
- note added: "Power"
- moved on the sheet: A101, D101, J101, J102, J103, J104, J105, J106, J107, J109, J110, J111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
