File: hardware/presto-jr-v2.0/regulators.kicad_sch (KiCad schematic)
At the start: 1 part

Commit message: updated v2
Changed lines of the file:
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@@
 			)
 		)
-		(property "Value" "GND"
-			(at 66.04 64.77 0)
+		(property "Value" "GND_LED"
+			(at 68.58 60.9599 0)
 			(show_name no)
 			(do_not_autoplace no)
@@
 					(size 1.27 1.27)
 				)
+				(justify left)
 			)
 		)
